File: hardware/main.sch (EAGLE design)
At the start: 8 parts, among them IC1 VNH3SP30, IC2 VNH3SP30, IC3 ATMEGA644A

Commit message: hurr durr
Parts:
- removed IC1, IC2: VNH3SP30, st-microelectronics:VNH3SP30
- added C4, C5: (no value), SparkFun:CAP0603-CAP
- added J1: AVR_SPI_PRG_6PTH, SparkFun:AVR_SPI_PRG_6PTH
- added JP1, JP3, JP4, JP6: M01, SparkFun:M01-SMTSO-256-ET
- added JP2, JP5: M01-SMTSO-256-ET, SparkFun:M01-SMTSO-256-ET
- added R1, R10, R11, R12, R13, R14, R15, R16, R17, R18, R19, R2, R20, R21, R3, R4, R5, R6, R7, R8, R9: (no value), SparkFun:RESISTOR0603-RES
- added S1: (no value), SparkFun:TAC_SWITCHSMD
- added U$4, U$6: VNH2SP30, SparkFun:VNH2SP30
Connections:
- new net 5V: IC3.VCC, IC3.VCC@1, IC3.VCC@2, J1.2, R7.2, U$1.VCC
- new net ACS712_OUT: U$1.VOUT
- new net CS1: C4.1, R1.2
- new net CS2: C5.1, R16.2
- new net DIAA1: R10.2
- new net DIAA2: R13.2
- new net DIAB1: R9.2
- new net DIAB2: R8.2
- new net INA1: R5.2
- new net INA2: R20.2
- new net INB1: R6.2
- new net INB2: R21.2
- new net MISO: IC3.(PCINT14/MISO)PB6, J1.1
- new net MOSI: IC3.(PCINT13/MOSI)PB5, J1.4
- new net N$10: R6.1, U$4.INB
- new net N$11: R15.1, R8.1, U$6.EN/DIAB
- new net N$12: R13.1, R14.1, U$6.EN/DIAA
- new net N$13: JP3.1, U$6.OUTA@1, U$6.OUTA@25, U$6.OUTA@30, U$6.OUTA@SLUG3
- new net N$14: JP4.1, U$6.OUTB@15, U$6.OUTB@16, U$6.OUTB@21, U$6.OUTB@SLUG2
- new net N$15: R12.1, R9.1, U$4.EN/DIAB
- new net N$16: R10.1, R11.1, U$4.EN/DIAA
- new net N$17: R16.1, R17.2, U$6.CS
- new net N$18: R18.1, U$6.PWM
- new net N$19: R20.1, U$6.INA
- new net N$20: R21.1, U$6.INB
- new net N$4: JP1.1, U$4.OUTA@1, U$4.OUTA@25, U$4.OUTA@30, U$4.OUTA@SLUG3
- new net N$5: JP6.1, U$4.OUTB@15, U$4.OUTB@16, U$4.OUTB@21, U$4.OUTB@SLUG2
- new net N$6: R1.1, R2.2, U$4.CS
- new net N$7: R3.1, U$4.PWM
- new net N$8: R5.1, U$4.INA
- new net N$9: JP2.1, U$1.IP-@3, U$1.IP-@4
- new net PWM1: R3.2, R4.2
- new net PWM2: R18.2, R19.2
- new net RESET: IC3.RESET, J1.5, R7.1, S1.1, S1.2
- new net SCK: IC3.(PCINT15/SCK)PB7, J1.3
- new net VCC: R11.2, R12.2, R14.2, R15.2, U$1.IP+@1, U$1.IP+@2, U$4.VCC@13, U$4.VCC@23, U$4.VCC@3, U$4.VCC@SLUG1, U$6.VCC@13, U$6.VCC@23, U$6.VCC@3, U$6.VCC@SLUG1
- net GND: now also C1.2, C4.2, C5.2, IC3.GND, IC3.GND@1, IC3.GND@2, IC3.GND@3, J1.6, JP5.1, R17.1, R19.1, R2.1, R4.1, S1.3, S1.4, U$1.GND, U$4.GNDA@26, U$4.GNDA@27, U$4.GNDA@28, U$4.GNDB@18, U$4.GNDB@19, U$4.GNDB@20, U$6.GNDA@26, U$6.GNDA@27, U$6.GNDA@28, U$6.GNDB@18, U$6.GNDB@19, U$6.GNDB@20
Other:
- moved on the sheet: C1, C2, C3, IC3, Q1, U$1

Commit message: blah
Parts:
- added IC1: 7805DT, linear:7805DT
- added LM3940(SOT223): LM3940 SOT223, LM3940:LM3940IMP-3.3
- added U1: (no value), adafruit:TXB0108PWR
- added XB2: XBEE-PRO, maxstream:XBEE-PRO
Connections:
- new net +3V3: LM3940(SOT223).OUT
- new net RXD: IC3.(PCINT24/RXD0)PD0, XB2.DOUT
- new net TXD: IC3.(PCINT25/TXD0)PD1, XB2.DIN/!CONFIG
- net 5V: now also IC1.VO
- net GND: now also IC1.GND, LM3940(SOT223).GND
- net VCC: now also IC1.VI, LM3940(SOT223).IN
Changed lines of the file:
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@@
 <?xml version="1.0" encoding="utf-8"?>
 <!DOCTYPE eagle SYSTEM "eagle.dtd">
-<eagle version="6.2">
+<eagle version="6.5.0">
 <drawing>
 <settings>
@@
 <layer number="54" name="bGND_GNDA" color="1" fill="9" visible="no" active="no"/>
 <layer number="56" name="wert" color="7" fill="1" visible="no" active="no"/>
+<layer number="57" name="tCAD" color="7" fill="1" visible="no" active="no"/>
 <layer number="91" name="Nets" color="2" fill="1" visible="yes" active="yes"/>
 <layer number="92" name="Busses" color="1" fill="1" visible="yes" active="yes"/>
@@
 <layer number="106" name="bPlate" color="7" fill="1" visible="no" active="yes"/>
 <layer number="107" name="Crop" color="7" fill="1" visible="no" active="yes"/>
+<layer number="108" name="fp8" color="7" fill="1" visible="no" active="yes"/>
+<layer number="109" name="fp9" color="7" fill="1" visible="no" active="yes"/>
+<layer number="110" name="fp0" color="7" fill="1" visible="no" active="yes"/>
+<layer number="111" name="LPC17xx" color="7" fill="1" visible="yes" active="yes"/>
+<layer number="112" name="tSilk" color="7" fill="1" visible="yes" active="yes"/>
 <layer number="116" name="Patch_BOT" color="9" fill="4" visible="no" active="yes"/>
 <layer number="121" name="_tsilk" color="7" fill="1" visible="no" active="yes"/>
 <layer number="122" name="_bsilk" color="7" fill="1" visible="no" active="yes"/>
+<layer number="123" name="tTestmark" color="7" fill="1" visible="no" active="yes"/>
+<layer number="124" name="bTestmark" color="7" fill="1" visible="no" active="yes"/>
 <layer number="125" name="_tNames" color="7" fill="1" visible="no" active="yes"/>
+<layer number="126" name="_bNames" color="7" fill="1" visible="yes" active="yes"/>
+<layer number="127" name="_tValues" color="7" fill="1" visible="yes" active="yes"/>
+<layer number="128" name="_bValues" color="7" fill="1" visible="yes" active="yes"/>
+<layer number="131" name="tAdjust" color="7" fill="1" visible="no" active="yes"/>
+<layer number="132" name="bAdjust" color="7" fill="1" visible="no" active="yes"/>
 <layer number="144" name="Drill_legend" color="7" fill="1" visible="no" active="yes"/>
+<layer number="150" name="Notes" color="7" fill="1" visible="no" active="yes"/>
 <layer number="151" name="HeatSink" color="7" fill="1" visible="no" active="yes"/>
+<layer number="152" name="_bDocu" color="7" fill="1" visible="yes" active="yes"/>
+<layer number="153" name="FabDoc1" color="6" fill="1" visible="no" active="no"/>
+<layer number="154" name="FabDoc2" color="2" fill="1" visible="no" active="no"/>
+<layer number="155" name="FabDoc3" color="7" fill="15" visible="no" active="no"/>
+<layer number="199" name="Contour" color="7" fill="1" visible="yes" active="yes"/>
 <layer number="200" name="200bmp" color="1" fill="10" visible="no" active="yes"/>
 <layer number="201" name="201bmp" color="2" fill="10" visible="no" active="yes"/>
@@
 <layer number="223" name="223bmp" color="24" fill="1" visible="no" active="no"/>
 <layer number="224" name="224bmp" color="25" fill="1" visible="no" active="no"/>
+<layer number="248" name="Housing" color="7" fill="1" visible="yes" active="yes"/>
+<layer number="249" name="Edge" color="7" fill="1" visible="yes" active="yes"/>
 <layer number="250" name="Descript" color="3" fill="1" visible="no" active="no"/>
 <layer number="251" name="SMDround" color="12" fill="11" visible="no" active="no"/>
@@
 <part name="R20" library="SparkFun" deviceset="RESISTOR" device="0603-RES"/>
 <part name="R21" library="SparkFun" deviceset="RESISTOR" device="0603-RES"/>
+<part name="XB2" library="maxstream" deviceset="XBEE" device="-PRO"/>
+<part name="U1" library="adafruit" deviceset="TXB0108PWR" device=""/>
+<part name="LM3940(SOT223)" library="LM3940" deviceset="LM3940IMP-3.3" device="" value="LM3940 SOT223"/>
+<part name="IC1" library="linear" deviceset="78*" device="DT" technology="05"/>
+<part name="P+6" library="SparkFun" deviceset="VCC" device=""/>
+<part name="P+7" library="SparkFun" deviceset="VCC" device=""/>
+<part name="U$7" library="SparkFun" deviceset="5V" device=""/>
+<part name="+3V1" library="supply1" deviceset="+3V3" device=""/>
+<part name="GND12" library="SparkFun" deviceset="GND" device=""/>
+<part name="GND13" library="SparkFun" deviceset="GND" device=""/>
 </parts>
 <sheets>
@@
 <instance part="R20" gate="G$1" x="127" y="35.56" rot="R180"/>
 <instance part="R21" gate="G$1" x="127" y="30.48" rot="R180"/>
+<instance part="XB2" gate="G$1" x="-129.54" y="48.26" rot="MR0"/>
+<instance part="U1" gate="G$1" x="22.86" y="170.18"/>
+<instance part="LM3940(SOT223)" gate="G$1" x="-182.88" y="-27.94"/>
+<instance part="IC1" gate="A1" x="-226.06" y="-30.48"/>
+<instance part="P+6" gate="1" x="-243.84" y="-25.4"/>
+<instance part="P+7" gate="1" x="-193.04" y="-25.4"/>
+<instance part="U$7" gate="G$1" x="-208.28" y="-25.4"/>
+<instance part="+3V1" gate="G$1" x="-147.32" y="-22.86"/>
+<instance part="GND12" gate="1" x="-226.06" y="-53.34"/>
+<instance part="GND13" gate="1" x="-170.18" y="-53.34"/>
 </instances>
 <busses>
@@
 <pinref part="GND11" gate="1" pin="GND"/>
 </segment>
+<segment>
+<pinref part="GND13" gate="1" pin="GND"/>
+<pinref part="LM3940(SOT223)" gate="G$1" pin="GND"/>
+<wire x1="-170.18" y1="-50.8" x2="-170.18" y2="-45.72" width="0.1524" layer="91"/>
+</segment>
+<segment>
+<pinref part="GND12" gate="1" pin="GND"/>
+<pinref part="IC1" gate="A1" pin="GND"/>
+<wire x1="-226.06" y1="-50.8" x2="-226.06" y2="-38.1" width="0.1524" layer="91"/>
+</segment>
 </net>
 <net name="VCC" class="0">
@@
 <junction x="170.18" y="63.5"/>
 </segment>
+<segment>
+<pinref part="P+7" gate="1" pin="VCC"/>
+<wire x1="-193.04" y1="-25.4" x2="-193.04" y2="-30.48" width="0.1524" layer="91"/>
+<pinref part="LM3940(SOT223)" gate="G$1" pin="IN"/>
+<wire x1="-193.04" y1="-30.48" x2="-185.42" y2="-30.48" width="0.1524" layer="91"/>
+</segment>
+<segment>
+<pinref part="P+6" gate="1" pin="VCC"/>
+<wire x1="-243.84" y1="-25.4" x2="-243.84" y2="-30.48" width="0.1524" layer="91"/>
+<pinref part="IC1" gate="A1" pin="VI"/>
+<wire x1="-243.84" y1="-30.48" x2="-236.22" y2="-30.48" width="0.1524" layer="91"/>
+</segment>
 </net>
 <net name="5V" class="0">
@@
 <pinref part="U$5" gate="G$1" pin="5V"/>
 <wire x1="-220.98" y1="193.04" x2="-220.98" y2="190.5" width="0.1524" layer="91"/>
+</segment>
+<segment>
+<pinref part="IC1" gate="A1" pin="VO"/>
+<wire x1="-215.9" y1="-30.48" x2="-208.28" y2="-30.48" width="0.1524" layer="91"/>
+<pinref part="U$7" gate="G$1" pin="5V"/>
+<wire x1="-208.28" y1="-30.48" x2="-208.28" y2="-25.4" width="0.1524" layer="91"/>
 </segment>
 </net>
@@
 </segment>
 </net>
+<net name="TXD" class="0">
+<segment>
+<pinref part="IC3" gate="G$1" pin="(PCINT25/TXD0)PD1"/>
+<wire x1="-96.52" y1="111.76" x2="-88.9" y2="111.76" width="0.1524" layer="91"/>
+<label x="-93.98" y="111.76" size="1.778" layer="95"/>
+</segment>
+<segment>
+<pinref part="XB2" gate="G$1" pin="DIN/!CONFIG"/>
+<wire x1="-114.3" y1="58.42" x2="-106.68" y2="58.42" width="0.1524" layer="91"/>
+<label x="-111.76" y="58.42" size="1.778" layer="95"/>
+</segment>
+</net>
+<net name="RXD" class="0">
+<segment>
+<pinref part="IC3" gate="G$1" pin="(PCINT24/RXD0)PD0"/>
+<wire x1="-96.52" y1="109.22" x2="-88.9" y2="109.22" width="0.1524" layer="91"/>
+<label x="-93.98" y="109.22" size="1.778" layer="95"/>
+</segment>
+<segment>
+<pinref part="XB2" gate="G$1" pin="DOUT"/>
+<wire x1="-114.3" y1="55.88" x2="-106.68" y2="55.88" width="0.1524" layer="91"/>
+<label x="-111.76" y="55.88" size="1.778" layer="95"/>
+</segment>
+</net>
+<net name="+3V3" class="0">
+<segment>
+<pinref part="LM3940(SOT223)" gate="G$1" pin="OUT"/>
+<wire x1="-154.94" y1="-30.48" x2="-147.32" y2="-30.48" width="0.1524" layer="91"/>
+<pinref part="+3V1" gate="G$1" pin="+3V3"/>
+<wire x1="-147.32" y1="-30.48" x2="-147.32" y2="-25.4" width="0.1524" layer="91"/>
+</segment>
+</net>

Commit message: blah
Connections:
- net +3V3: now also U1.VCCA
- net 5V: now also U1.VCCB
- net GND: now also U1.GND
Other:
- moved on the sheet: U1
Changed lines of the file:
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@@
 <part name="GND12" library="SparkFun" deviceset="GND" device=""/>
 <part name="GND13" library="SparkFun" deviceset="GND" device=""/>
+<part name="+3V2" library="supply1" deviceset="+3V3" device=""/>
+<part name="U$8" library="SparkFun" deviceset="5V" device=""/>
+<part name="GND14" library="SparkFun" deviceset="GND" device=""/>
 </parts>
 <sheets>
@@
 <instance part="C3" gate="G$1" x="-170.18" y="162.56"/>
 <instance part="GND1" gate="1" x="-177.8" y="152.4"/>
-<instance part="U$2" gate="G$1" x="-152.4" y="198.12"/>
+<instance part="U$2" gate="G$1" x="-152.4" y="203.2"/>
 <instance part="GND3" gate="1" x="-152.4" y="104.14"/>
 <instance part="U$3" gate="G$1" x="-203.2" y="76.2"/>
@@
 <instance part="R21" gate="G$1" x="127" y="30.48" rot="R180"/>
 <instance part="XB2" gate="G$1" x="-129.54" y="48.26" rot="MR0"/>
-<instance part="U1" gate="G$1" x="22.86" y="170.18"/>
+<instance part="U1" gate="G$1" x="-35.56" y="180.34"/>
 <instance part="LM3940(SOT223)" gate="G$1" x="-182.88" y="-27.94"/>
 <instance part="IC1" gate="A1" x="-226.06" y="-30.48"/>
@@
 <instance part="GND12" gate="1" x="-226.06" y="-53.34"/>
 <instance part="GND13" gate="1" x="-170.18" y="-53.34"/>
+<instance part="+3V2" gate="G$1" x="-38.1" y="205.74"/>
+<instance part="U$8" gate="G$1" x="-33.02" y="203.2"/>
+<instance part="GND14" gate="1" x="-35.56" y="152.4"/>
 </instances>
 <busses>
@@
 <wire x1="-226.06" y1="-50.8" x2="-226.06" y2="-38.1" width="0.1524" layer="91"/>
 </segment>
+<segment>
+<pinref part="U1" gate="G$1" pin="GND"/>
+<pinref part="GND14" gate="1" pin="GND"/>
+<wire x1="-35.56" y1="154.94" x2="-35.56" y2="157.48" width="0.1524" layer="91"/>
+</segment>
 </net>
 <net name="VCC" class="0">
@@
 <wire x1="-149.86" y1="193.04" x2="-152.4" y2="193.04" width="0.1524" layer="91"/>
 <wire x1="-152.4" y1="193.04" x2="-152.4" y2="195.58" width="0.1524" layer="91"/>
-<wire x1="-152.4" y1="195.58" x2="-152.4" y2="198.12" width="0.1524" layer="91"/>
+<wire x1="-152.4" y1="195.58" x2="-152.4" y2="203.2" width="0.1524" layer="91"/>
 <junction x="-152.4" y="195.58"/>
 <pinref part="U$2" gate="G$1" pin="5V"/>
@@
 <pinref part="U$7" gate="G$1" pin="5V"/>
 <wire x1="-208.28" y1="-30.48" x2="-208.28" y2="-25.4" width="0.1524" layer="91"/>
+</segment>
+<segment>
+<pinref part="U$8" gate="G$1" pin="5V"/>
+<pinref part="U1" gate="G$1" pin="VCCB"/>
+<wire x1="-33.02" y1="203.2" x2="-33.02" y2="200.66" width="0.1524" layer="91"/>
 </segment>
 </net>
@@
 <wire x1="-147.32" y1="-30.48" x2="-147.32" y2="-25.4" width="0.1524" layer="91"/>
 </segment>
-</net>
+<segment>
+<pinref part="+3V2" gate="G$1" pin="+3V3"/>
+<pinref part="U1" gate="G$1" pin="VCCA"/>
+<wire x1="-38.1" y1="203.2" x2="-38.1" y2="200.66" width="0.1524" layer="91"/>
+</segment>
+</net>

Commit message: Duh
Parts:
- added C6, C7, C8: (no value), adafruit:CPOL-US140CLH-1010
Connections:
- net 5V: now also LM3940(SOT223).IN
- net VCC: no longer LM3940(SOT223).IN
Changed lines of the file:
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@@
 <part name="IC1" library="linear" deviceset="78*" device="DT" technology="05"/>
 <part name="P+6" library="SparkFun" deviceset="VCC" device=""/>
-<part name="P+7" library="SparkFun" deviceset="VCC" device=""/>
 <part name="U$7" library="SparkFun" deviceset="5V" device=""/>
 <part name="+3V1" library="supply1" deviceset="+3V3" device=""/>
@@
 <part name="U$8" library="SparkFun" deviceset="5V" device=""/>
 <part name="GND14" library="SparkFun" deviceset="GND" device=""/>
+<part name="C6" library="adafruit" deviceset="CPOL-US" device="140CLH-1010"/>
+<part name="C7" library="adafruit" deviceset="CPOL-US" device="140CLH-1010"/>
+<part name="C8" library="adafruit" deviceset="CPOL-US" device="140CLH-1010"/>
+<part name="U$9" library="SparkFun" deviceset="5V" device=""/>
 </parts>
 <sheets>
@@
 <instance part="IC1" gate="A1" x="-226.06" y="-30.48"/>
 <instance part="P+6" gate="1" x="-243.84" y="-25.4"/>
-<instance part="P+7" gate="1" x="-193.04" y="-25.4"/>
 <instance part="U$7" gate="G$1" x="-208.28" y="-25.4"/>
 <instance part="+3V1" gate="G$1" x="-147.32" y="-22.86"/>
@@
 <instance part="U$8" gate="G$1" x="-33.02" y="203.2"/>
 <instance part="GND14" gate="1" x="-35.56" y="152.4"/>
+<instance part="C6" gate="G$1" x="-243.84" y="-40.64"/>
+<instance part="C7" gate="G$1" x="-208.28" y="-43.18"/>
+<instance part="C8" gate="G$1" x="-144.78" y="-40.64"/>
+<instance part="U$9" gate="G$1" x="-193.04" y="-25.4"/>
 </instances>
 <busses>
@@
 </segment>
 <segment>
-<pinref part="P+7" gate="1" pin="VCC"/>
-<wire x1="-193.04" y1="-25.4" x2="-193.04" y2="-30.48" width="0.1524" layer="91"/>
-<pinref part="LM3940(SOT223)" gate="G$1" pin="IN"/>
-<wire x1="-193.04" y1="-30.48" x2="-185.42" y2="-30.48" width="0.1524" layer="91"/>
-</segment>
-<segment>
 <pinref part="P+6" gate="1" pin="VCC"/>
 <wire x1="-243.84" y1="-25.4" x2="-243.84" y2="-30.48" width="0.1524" layer="91"/>
@@
 </segment>
 <segment>
-<pinref part="IC1" gate="A1" pin="VO"/>
-<wire x1="-215.9" y1="-30.48" x2="-208.28" y2="-30.48" width="0.1524" layer="91"/>
-<pinref part="U$7" gate="G$1" pin="5V"/>
-<wire x1="-208.28" y1="-30.48" x2="-208.28" y2="-25.4" width="0.1524" layer="91"/>
-</segment>
-<segment>
 <pinref part="U$8" gate="G$1" pin="5V"/>
 <pinref part="U1" gate="G$1" pin="VCCB"/>
 <wire x1="-33.02" y1="203.2" x2="-33.02" y2="200.66" width="0.1524" layer="91"/>
 </segment>
-</net>
+<segment>
+<pinref part="U$7" gate="G$1" pin="5V"/>
+<wire x1="-208.28" y1="-25.4" x2="-208.28" y2="-30.48" width="0.1524" layer="91"/>
+<pinref part="IC1" gate="A1" pin="VO"/>
+<wire x1="-208.28" y1="-30.48" x2="-215.9" y2="-30.48" width="0.1524" layer="91"/>
+</segment>
+<segment>
+<pinref part="U$9" gate="G$1" pin="5V"/>
+<wire x1="-193.04" y1="-25.4" x2="-193.04" y2="-30.48" width="0.1524" layer="91"/>
+<pinref part="LM3940(SOT223)" gate="G$1" pin="IN"/>
+<wire x1="-193.04" y1="-30.48" x2="-185.42" y2="-30.48" width="0.1524" layer="91"/>
+</segment>
+</net>

Commit message: Better IO
Parts:
- removed JP1, JP3, JP4, JP6: M01, SparkFun:M01-SMTSO-256-ET
- removed JP2, JP5: M01-SMTSO-256-ET, SparkFun:M01-SMTSO-256-ET
- added GPS: (no value), con-amp:MTA04-100
- added I2C: (no value), con-amp:MTA05-100
- added J2: 350792-1, con-amp:350792-1
- added J3: 350428-1, con-amp:350428-1
Connections:
- removed net N$13: JP3.1, U$6.OUTA@1, U$6.OUTA@25, U$6.OUTA@30, U$6.OUTA@SLUG3
- removed net N$14: JP4.1, U$6.OUTB@15, U$6.OUTB@16, U$6.OUTB@21, U$6.OUTB@SLUG2
- removed net N$4: JP1.1, U$4.OUTA@1, U$4.OUTA@25, U$4.OUTA@30, U$4.OUTA@SLUG3
- removed net N$5: JP6.1, U$4.OUTB@15, U$4.OUTB@16, U$4.OUTB@21, U$4.OUTB@SLUG2
- removed net RXD: IC3.(PCINT24/RXD0)PD0, XB2.DOUT
- removed net TXD: IC3.(PCINT25/TXD0)PD1, XB2.DIN/!CONFIG
- new net GPS_RX: GPS.2
- new net GPS_TX: GPS.3
- new net OUTA1: J2.1, U$4.OUTA@1, U$4.OUTA@25, U$4.OUTA@30, U$4.OUTA@SLUG3
- new net OUTA2: J2.3, U$6.OUTA@1, U$6.OUTA@25, U$6.OUTA@30, U$6.OUTA@SLUG3
- new net OUTB1: J2.2, U$4.OUTB@15, U$4.OUTB@16, U$4.OUTB@21, U$4.OUTB@SLUG2
- new net OUTB2: J2.4, U$6.OUTB@15, U$6.OUTB@16, U$6.OUTB@21, U$6.OUTB@SLUG2
- new net SCL: I2C.1, IC3.(PCINT16/SCL)PC0
- new net SDA: I2C.2, IC3.(PCINT17/SDA)PC1
- net +3V3: now also GPS.1, I2C.3, XB2.VCC
- net 5V: now also I2C.4
- net GND: now also GPS.4, I2C.5, J3.1, XB2.GND; no longer JP5.1
- net N$9: now also J3.2; no longer JP2.1
Other:
- moved on the sheet: C6, C8

Commit message: More improvements
Parts:
- added C9: (no value), SparkFun:CAP0603-CAP
- C7, C8: device adafruit:CPOL-US140CLH-1010 -> SparkFun:CAP0603-CAP
Connections:
- new net RX: U1.A2, XB2.DOUT
- new net RXD: IC3.(PCINT24/RXD0)PD0, U1.B2
- new net TX: U1.A1, XB2.DIN/!CONFIG
- new net TXD: IC3.(PCINT25/TXD0)PD1, U1.B1
- net +3V3: now also C8.2, XB2.VREF; no longer I2C.3
- net 5V: now also C7.2, I2C.3; no longer I2C.4
- net GND: now also C6.-, C7.1, C8.1, C9.1
- net INA1: now also IC3.(PCINT23/TOSC2)PC7
- net INA2: now also IC3.(PCINT22/TOSC1)PC6
- net INB1: now also IC3.(PCINT21/TDI)PC5
- net INB2: now also IC3.(PCINT20/TDO)PC4
- net PWM1: now also IC3.(PCINT31/OC2A)PD7
- net PWM2: now also IC3.(PCINT30/OC2B/ICP)PD6
- net VCC: now also C6.+, C9.2
Other:
- moved on the sheet: C2, C6
